Commit message: Add tf fixes

File: models/autonomous_vehicle/model.urdf (robot description, URDF)
Before this commit: robot autonomous_vehicle, 13 links, 12 joints
Links:
- link chassis: geometry collision box size=0.7 0.35 0.12; visual box size=0.7 0.32 0.12
- link front_axle: geometry visual cylinder length=0.44 radius=0.02
Joints:
- joint front_left_wheel_joint: origin xyz=0 0.07 0 rpy=-1.5707 0 0 -> xyz=0 0.04 0 rpy=-1.5707 0 0
- joint front_left_wheel_steering_joint: origin xyz=0 0.19 0 rpy=0 0 0 -> xyz=0 0.22 0 rpy=0 0 0
- joint front_right_wheel_joint: origin xyz=0 -0.07 0 rpy=-1.5707 0 0 -> xyz=0 -0.04 0 rpy=-1.5707 0 0
- joint front_right_wheel_steering_joint: origin xyz=0 -0.19 0 rpy=0 0 0 -> xyz=0 -0.22 0 rpy=0 0 0
- joint stereo_camera_holder_joint: origin xyz=0.3 0 0.15 rpy=0 0 0 -> xyz=0.3 0 0.25 rpy=0 0 0

Commit message: Implement sensor fusion with robot_localization

File: models/autonomous_vehicle/model.urdf (robot description, URDF)
Before this commit: robot autonomous_vehicle, 13 links, 12 joints
Links:
- added link imu_sensor, mass 0.1; visual sphere radius=0.02
Joints:
- added joint imu_sensor_joint: type fixed, parent chassis, child imu_sensor, origin xyz=0.32 0 0.08 rpy=0 0 0

Commit message: Nav2 adaptation progress

File: models/autonomous_vehicle/model.urdf (robot description, URDF)
Before this commit: robot autonomous_vehicle, 14 links, 13 joints
Links:
- added link base_footprint
Joints:
- removed joint dummy_base_link_joint
- added joint dummy_chassis_joint: type fixed, parent base_link, child chassis
- added joint footprint_joint: type fixed, parent base_link, child base_footprint, origin xyz=0.0 0.0 -0.1 rpy=0 0 0

Commit message: Add navigation progress

File: models/autonomous_vehicle/model.urdf (robot description, URDF)
Before this commit: robot autonomous_vehicle, 15 links, 14 joints
Links:
- link chassis: geometry collision box size=0.7 0.25 0.12; visual box size=0.7 0.25 0.12
Joints:
- joint rear_left_wheel_joint: limit lower=-3.1416 upper=3.1416 effort=25 velocity=10.0 -> (none); type revolute -> continuous

Commit message: Add sonar sensors and fix architecture

File: models/autonomous_vehicle/model.urdf (robot description, URDF)
Before this commit: robot autonomous_vehicle, 15 links, 14 joints
Links:
- added link front_bumper_center, mass 0.3; collision box size=0.03 0.34 0.07; visual box size=0.03 0.34 0.07
- added link front_bumper_left, mass 0.2; collision box size=0.03 0.14 0.07; visual box size=0.03 0.14 0.07
- added link front_bumper_right, mass 0.2; collision box size=0.03 0.14 0.07; visual box size=0.03 0.14 0.07
- added link left_side_bumper, mass 0.15; collision box size=0.32 0.03 0.07; visual box size=0.32 0.03 0.07
- added link rear_bumper_center, mass 0.3; collision box size=0.03 0.34 0.07; visual box size=0.03 0.34 0.07
- added link rear_bumper_left, mass 0.2; collision box size=0.03 0.14 0.07; visual box size=0.03 0.14 0.07
- added link rear_bumper_right, mass 0.2; collision box size=0.03 0.14 0.07; visual box size=0.03 0.14 0.07
- added link right_side_bumper, mass 0.15; collision box size=0.32 0.03 0.07; visual box size=0.32 0.03 0.07
- added link sonar_front_bumper_center, mass 0.05; collision cylinder length=0.02 radius=0.015; visual cylinder length=0.02 radius=0.015
- added link sonar_front_bumper_left, mass 0.05; collision cylinder length=0.02 radius=0.015; visual cylinder length=0.02 radius=0.015
- added link sonar_front_bumper_right, mass 0.05; collision cylinder length=0.02 radius=0.015; visual cylinder length=0.02 radius=0.015
- added link sonar_left_side_bumper, mass 0.05; collision cylinder length=0.02 radius=0.015; visual cylinder length=0.02 radius=0.015
- added link sonar_rear_bumper_center, mass 0.05; collision cylinder length=0.02 radius=0.015; visual cylinder length=0.02 radius=0.015
- added link sonar_rear_bumper_left, mass 0.05; collision cylinder length=0.02 radius=0.015; visual cylinder length=0.02 radius=0.015
- added link sonar_rear_bumper_right, mass 0.05; collision cylinder length=0.02 radius=0.015; visual cylinder length=0.02 radius=0.015
- added link sonar_right_side_bumper, mass 0.05; collision cylinder length=0.02 radius=0.015; visual cylinder length=0.02 radius=0.015
Joints:
- added joint front_bumper_center_joint: type fixed, parent chassis, child front_bumper_center, origin xyz=0.49 0 0 rpy=0 0 0
- added joint front_bumper_left_joint: type fixed, parent chassis, child front_bumper_left, origin xyz=0.4719 0.2376 0 rpy=0 0 0.2618
- added joint front_bumper_right_joint: type fixed, parent chassis, child front_bumper_right, origin xyz=0.4719 -0.2376 0 rpy=0 0 -0.2618
- added joint left_side_bumper_joint: type fixed, parent chassis, child left_side_bumper, origin xyz=0.0 0.295 0 rpy=0 0 0
- added joint rear_bumper_center_joint: type fixed, parent chassis, child rear_bumper_center, origin xyz=-0.49 0 0 rpy=0 0 0
- added joint rear_bumper_left_joint: type fixed, parent chassis, child rear_bumper_left, origin xyz=-0.4719 0.2376 0 rpy=0 0 -0.2618
- added joint rear_bumper_right_joint: type fixed, parent chassis, child rear_bumper_right, origin xyz=-0.4719 -0.2376 0 rpy=0 0 0.2618
- added joint right_side_bumper_joint: type fixed, parent chassis, child right_side_bumper, origin xyz=0.0 -0.295 0 rpy=0 0 0
- added joint sonar_front_bumper_center_joint: type fixed, parent front_bumper_center, child sonar_front_bumper_center, origin xyz=0.02 0 0 rpy=0 0 0
- added joint sonar_front_bumper_left_joint: type fixed, parent front_bumper_left, child sonar_front_bumper_left, origin xyz=0.02 0 0 rpy=0 0 0
- added joint sonar_front_bumper_right_joint: type fixed, parent front_bumper_right, child sonar_front_bumper_right, origin xyz=0.02 0 0 rpy=0 0 0
- added joint sonar_left_side_bumper_joint: type fixed, parent left_side_bumper, child sonar_left_side_bumper, origin xyz=0 0.02 0 rpy=0 0 1.5707
- added joint sonar_rear_bumper_center_joint: type fixed, parent rear_bumper_center, child sonar_rear_bumper_center, origin xyz=-0.02 0 0 rpy=0 0 3.1416
- added joint sonar_rear_bumper_left_joint: type fixed, parent rear_bumper_left, child sonar_rear_bumper_left, origin xyz=-0.02 0 0 rpy=0 0 3.1416
- added joint sonar_rear_bumper_right_joint: type fixed, parent rear_bumper_right, child sonar_rear_bumper_right, origin xyz=-0.02 0 0 rpy=0 0 3.1416
- added joint sonar_right_side_bumper_joint: type fixed, parent right_side_bumper, child sonar_right_side_bumper, origin xyz=0 -0.02 0 rpy=0 0 -1.5707
- joint rear_left_wheel_joint: origin xyz=0 -0.26 0 rpy=-1.5707 0 0 -> xyz=0 0.26 0 rpy=-1.5707 0 0
- joint rear_right_wheel_joint: origin xyz=0 0.26 0 rpy=-1.5707 0 0 -> xyz=0 -0.26 0 rpy=-1.5707 0 0

Commit message: Refine pure pursuit and visual odometry integration

File: models/autonomous_vehicle/model.urdf (robot description, URDF)
Before this commit: robot autonomous_vehicle, 31 links, 30 joints
Joints:
- joint front_left_wheel_steering_joint: limit lower=-0.6 upper=0.6 effort=25 velocity=1.0 -> lower=-0.6 upper=0.6 effort=25 velocity=1.2
- joint front_right_wheel_steering_joint: limit lower=-0.6 upper=0.6 effort=25 velocity=1.0 -> lower=-0.6 upper=0.6 effort=25 velocity=1.2

Commit message: Fix frame alignment (WIP)

File: models/autonomous_vehicle/model.urdf (robot description, URDF)
Before this commit: robot autonomous_vehicle, 31 links, 30 joints
Joints:
- joint footprint_joint: child base_footprint -> base_link; origin xyz=0.0 0.0 -0.1 rpy=0 0 0 -> xyz=0.0 0.0 0.1 rpy=0 0 0; parent base_link -> base_footprint

Commit message: Update vehicle geometry and navigation params

File: models/autonomous_vehicle/model.urdf (robot description, URDF)
Before this commit: robot autonomous_vehicle, 31 links, 30 joints
Links:
- link chassis: geometry collision box size=0.7 0.2 0.0465108; visual box size=0.7 0.2 0.0465108
- link front_axle: geometry visual cylinder length=0.33 radius=0.02
- link front_bumper_center: geometry collision box size=0.015 0.14 0.04; visual box size=0.015 0.14 0.04
- link front_bumper_left: geometry collision box size=0.015 0.09 0.04; visual box size=0.015 0.09 0.04
- link front_bumper_right: geometry collision box size=0.015 0.09 0.04; visual box size=0.015 0.09 0.04
- link front_left_wheel: geometry collision cylinder length=0.058866 radius=0.085; visual cylinder length=0.058866 radius=0.085
- link front_right_wheel: geometry collision cylinder length=0.058866 radius=0.085; visual cylinder length=0.058866 radius=0.085
- link left_side_bumper: geometry collision box size=0.34 0.015 0.04; visual box size=0.34 0.015 0.04
- link rear_axle: geometry visual cylinder length=0.37 radius=0.02
- link rear_bumper_center: geometry collision box size=0.015 0.14 0.04; visual box size=0.015 0.14 0.04
- link rear_bumper_left: geometry collision box size=0.015 0.09 0.04; visual box size=0.015 0.09 0.04
- link rear_bumper_right: geometry collision box size=0.015 0.09 0.04; visual box size=0.015 0.09 0.04
- link rear_left_wheel: geometry collision cylinder length=0.058866 radius=0.085; visual cylinder length=0.058866 radius=0.085
- link rear_right_wheel: geometry collision cylinder length=0.058866 radius=0.085; visual cylinder length=0.058866 radius=0.085
- link right_side_bumper: geometry collision box size=0.34 0.015 0.04; visual box size=0.34 0.015 0.04
- link stereo_camera_holder: geometry collision box size=0.04 0.25 0.05; visual box size=0.04 0.25 0.05
Joints:
- joint footprint_joint: origin xyz=0.0 0.0 0.1 rpy=0 0 0 -> xyz=0.0 0.0 0.085 rpy=0 0 0
- joint front_axle_joint: origin xyz=0.3 0 0 rpy=0 0 0 -> xyz=0.28059 0 0 rpy=0 0 0
- joint front_bumper_center_joint: origin xyz=0.49 0 0 rpy=0 0 0 -> xyz=0.4483 0 0 rpy=0 0 0
- joint front_bumper_left_joint: origin xyz=0.4719 0.2376 0 rpy=0 0 0.2618 -> xyz=0.4187 0.1773 0 rpy=0 0 0.7854
- joint front_bumper_right_joint: origin xyz=0.4719 -0.2376 0 rpy=0 0 -0.2618 -> xyz=0.4187 -0.1773 0 rpy=0 0 -0.7854
- joint front_left_wheel_joint: origin xyz=0 0.04 0 rpy=-1.5707 0 0 -> xyz=0 0.02 0 rpy=-1.5707 0 0
- joint front_left_wheel_steering_joint: origin xyz=0 0.22 0 rpy=0 0 0 -> xyz=0 0.165 0 rpy=0 0 0
- joint front_right_wheel_joint: origin xyz=0 -0.04 0 rpy=-1.5707 0 0 -> xyz=0 -0.02 0 rpy=-1.5707 0 0
- joint front_right_wheel_steering_joint: origin xyz=0 -0.22 0 rpy=0 0 0 -> xyz=0 -0.165 0 rpy=0 0 0
- joint left_side_bumper_joint: origin xyz=0.0 0.295 0 rpy=0 0 0 -> xyz=0.0 0.2069 0 rpy=0 0 0
- joint rear_axle_joint: origin xyz=-0.3 0 0 rpy=0 0 0 -> xyz=-0.28059 0 0 rpy=0 0 0
- joint rear_bumper_center_joint: origin xyz=-0.49 0 0 rpy=0 0 0 -> xyz=-0.4483 0 0 rpy=0 0 0
- joint rear_bumper_left_joint: origin xyz=-0.4719 0.2376 0 rpy=0 0 -0.2618 -> xyz=-0.4187 0.1773 0 rpy=0 0 -0.7854
- joint rear_bumper_right_joint: origin xyz=-0.4719 -0.2376 0 rpy=0 0 0.2618 -> xyz=-0.4187 -0.1773 0 rpy=0 0 0.7854
- joint rear_left_wheel_joint: origin xyz=0 0.26 0 rpy=-1.5707 0 0 -> xyz=0 0.185 0 rpy=-1.5707 0 0
- joint rear_right_wheel_joint: origin xyz=0 -0.26 0 rpy=-1.5707 0 0 -> xyz=0 -0.185 0 rpy=-1.5707 0 0
- joint right_side_bumper_joint: origin xyz=0.0 -0.295 0 rpy=0 0 0 -> xyz=0.0 -0.2069 0 rpy=0 0 0
- joint sonar_left_side_bumper_joint: origin xyz=0 0.02 0 rpy=0 0 1.5707 -> xyz=0 0.015 0 rpy=0 0 1.5707
- joint sonar_right_side_bumper_joint: origin xyz=0 -0.02 0 rpy=0 0 -1.5707 -> xyz=0 -0.015 0 rpy=0 0 -1.5707
- joint stereo_camera_holder_joint: origin xyz=0.3 0 0.25 rpy=0 0 0 -> xyz=0.21879 0 0.2578 rpy=0 0 0

Commit message: Revert "Update vehicle geometry and navigation params"
This reverts commit 4a2e66ca2ce120d81a9a41b4724c0ab9954034a7.

File: models/autonomous_vehicle/model.urdf (robot description, URDF)
Before this commit: robot autonomous_vehicle, 31 links, 30 joints
Links:
- link chassis: geometry collision box size=0.7 0.25 0.12; visual box size=0.7 0.25 0.12
- link front_axle: geometry visual cylinder length=0.44 radius=0.02
- link front_bumper_center: geometry collision box size=0.03 0.34 0.07; visual box size=0.03 0.34 0.07
- link front_bumper_left: geometry collision box size=0.03 0.14 0.07; visual box size=0.03 0.14 0.07
- link front_bumper_right: geometry collision box size=0.03 0.14 0.07; visual box size=0.03 0.14 0.07
- link front_left_wheel: geometry collision cylinder length=0.1 radius=0.1; visual cylinder length=0.1 radius=0.1
- link front_right_wheel: geometry collision cylinder length=0.1 radius=0.1; visual cylinder length=0.1 radius=0.1
- link left_side_bumper: geometry collision box size=0.32 0.03 0.07; visual box size=0.32 0.03 0.07
- link rear_axle: geometry visual cylinder length=0.52 radius=0.02
- link rear_bumper_center: geometry collision box size=0.03 0.34 0.07; visual box size=0.03 0.34 0.07
- link rear_bumper_left: geometry collision box size=0.03 0.14 0.07; visual box size=0.03 0.14 0.07
- link rear_bumper_right: geometry collision box size=0.03 0.14 0.07; visual box size=0.03 0.14 0.07
- link rear_left_wheel: geometry collision cylinder length=0.1 radius=0.1; visual cylinder length=0.1 radius=0.1
- link rear_right_wheel: geometry collision cylinder length=0.1 radius=0.1; visual cylinder length=0.1 radius=0.1
- link right_side_bumper: geometry collision box size=0.32 0.03 0.07; visual box size=0.32 0.03 0.07
- link stereo_camera_holder: geometry collision box size=0.04 0.25 0.06; visual box size=0.04 0.25 0.06
Joints:
- joint footprint_joint: origin xyz=0.0 0.0 0.085 rpy=0 0 0 -> xyz=0.0 0.0 0.1 rpy=0 0 0
- joint front_axle_joint: origin xyz=0.28059 0 0 rpy=0 0 0 -> xyz=0.3 0 0 rpy=0 0 0
- joint front_bumper_center_joint: origin xyz=0.4483 0 0 rpy=0 0 0 -> xyz=0.49 0 0 rpy=0 0 0
- joint front_bumper_left_joint: origin xyz=0.4187 0.1773 0 rpy=0 0 0.7854 -> xyz=0.4719 0.2376 0 rpy=0 0 0.2618
- joint front_bumper_right_joint: origin xyz=0.4187 -0.1773 0 rpy=0 0 -0.7854 -> xyz=0.4719 -0.2376 0 rpy=0 0 -0.2618
- joint front_left_wheel_joint: origin xyz=0 0.02 0 rpy=-1.5707 0 0 -> xyz=0 0.04 0 rpy=-1.5707 0 0
- joint front_left_wheel_steering_joint: origin xyz=0 0.165 0 rpy=0 0 0 -> xyz=0 0.22 0 rpy=0 0 0
- joint front_right_wheel_joint: origin xyz=0 -0.02 0 rpy=-1.5707 0 0 -> xyz=0 -0.04 0 rpy=-1.5707 0 0
- joint front_right_wheel_steering_joint: origin xyz=0 -0.165 0 rpy=0 0 0 -> xyz=0 -0.22 0 rpy=0 0 0
- joint left_side_bumper_joint: origin xyz=0.0 0.2069 0 rpy=0 0 0 -> xyz=0.0 0.295 0 rpy=0 0 0
- joint rear_axle_joint: origin xyz=-0.28059 0 0 rpy=0 0 0 -> xyz=-0.3 0 0 rpy=0 0 0
- joint rear_bumper_center_joint: origin xyz=-0.4483 0 0 rpy=0 0 0 -> xyz=-0.49 0 0 rpy=0 0 0
- joint rear_bumper_left_joint: origin xyz=-0.4187 0.1773 0 rpy=0 0 -0.7854 -> xyz=-0.4719 0.2376 0 rpy=0 0 -0.2618
- joint rear_bumper_right_joint: origin xyz=-0.4187 -0.1773 0 rpy=0 0 0.7854 -> xyz=-0.4719 -0.2376 0 rpy=0 0 0.2618
- joint rear_left_wheel_joint: origin xyz=0 0.185 0 rpy=-1.5707 0 0 -> xyz=0 0.26 0 rpy=-1.5707 0 0
- joint rear_right_wheel_joint: origin xyz=0 -0.185 0 rpy=-1.5707 0 0 -> xyz=0 -0.26 0 rpy=-1.5707 0 0
- joint right_side_bumper_joint: origin xyz=0.0 -0.2069 0 rpy=0 0 0 -> xyz=0.0 -0.295 0 rpy=0 0 0
- joint sonar_left_side_bumper_joint: origin xyz=0 0.015 0 rpy=0 0 1.5707 -> xyz=0 0.02 0 rpy=0 0 1.5707
- joint sonar_right_side_bumper_joint: origin xyz=0 -0.015 0 rpy=0 0 -1.5707 -> xyz=0 -0.02 0 rpy=0 0 -1.5707
- joint stereo_camera_holder_joint: origin xyz=0.21879 0 0.2578 rpy=0 0 0 -> xyz=0.3 0 0.25 rpy=0 0 0
